File: model-train-cdu/model-train-cdu.kicad_pcb (KiCad board)
At the start: 2 copper layers, 20 parts, among them J1 Screw_Terminal_01x16, J2 Screw_Terminal_01x12, J3 Screw_Terminal_01x12, J4 Screw_Terminal_01x16, Q1 TIP121

Commit message: add mfg files
Other:
- board outline added: 81.2 x 82.6 mm
- board text added: "JAB CDU v1"
Changed lines of the file:
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@@
   (general
     (thickness 1.6)
-    (drawings 0)
+    (drawings 5)
     (tracks 68)
     (zones 0)
@@
       (outputformat 1)
       (mirror false)
-      (drillshape 1)
+      (drillshape 0)
       (scaleselection 1)
-      (outputdirectory ""))
+      (outputdirectory "mfg"))
   )
   (net 0 "")
@@
     )
   )
+  (gr_text "JAB CDU v1" (at 81 -38) (layer F.SilkS)
+    (effects (font (size 2 2) (thickness 0.2)))
+  )
+  (gr_line (start 122 -58) (end 40.8 -58) (layer Edge.Cuts) (width 0.05))
+  (gr_line (start 122 24.6) (end 122 -58) (layer Edge.Cuts) (width 0.05))
+  (gr_line (start 40.8 24.6) (end 122 24.6) (layer Edge.Cuts) (width 0.05))
+  (gr_line (start 40.8 -58) (end 40.8 24.6) (layer Edge.Cuts) (width 0.05))
   (segment (start 80.4 -1.584) (end 80.4 -3.6) (width 1.016) (layer F.Cu) (net 1))
   (segment (start 88.8 3.8) (end 85.784 3.8) (width 1.016) (layer F.Cu) (net 1))
