File: cat-timer/cat-timer.sch (KiCad schematic (older format))
At the start: 8 parts

Commit message: add more comments
Parts:
- gave numbers to parts that had none: 8
Other:
- note added: "WiFi Timer is rated from 6-28V. 6V seems \nto be the absolute min -- it will not sink \nmuch curernt unless voltage at timer is \n6V or higher."
- note added: "use schottkey diode here \nif running from 6V lead acid\nbattery"
Changed lines of the file:
@@
 $EndDescr
 $Comp
-L bec-connector:xConnect_smd J?
+L bec-connector:xConnect_smd J1
 U 1 1 5F982B6C
 P 1800 3050
-F 0 "J?" H 1692 3243 50  0000 C CNN
+F 0 "J1" H 1692 3243 50  0000 C CNN
 F 1 "xConnect_smd" H 1692 3244 50  0001 C CNN
 F 2 "BEC:xConnect_smd" H 1750 2800 50  0001 C CNN
@@
 $EndComp
 $Comp
-L bec-connector:xConnect_smd J?
+L bec-connector:xConnect_smd J2
 U 1 1 5F984C64
 P 5850 3050
-F 0 "J?" H 5878 3030 50  0000 L CNN
+F 0 "J2" H 5878 3030 50  0000 L CNN
 F 1 "xConnect_smd" H 5878 2985 50  0001 L CNN
 F 2 "BEC:xConnect_smd" H 5800 2800 50  0001 C CNN
@@
 $EndComp
 $Comp
-L bec-interface:WiFiTimer U?
+L bec-interface:WiFiTimer U1
 U 1 1 5F986799
 P 4050 4150
-F 0 "U?" H 4568 4196 50  0000 L CNN
+F 0 "U1" H 4568 4196 50  0000 L CNN
 F 1 "WiFiTimer" H 4568 4105 50  0000 L CNN
 F 2 "" H 3600 3700 50  0001 C CNN
@@
 	2000 2950 2700 2950
 $Comp
-L Diode:1N914 D?
+L Diode:1N914 D1
 U 1 1 5F98A3D7
 P 2700 3300
-F 0 "D?" V 2746 3220 50  0000 R CNN
+F 0 "D1" V 2746 3220 50  0000 R CNN
 F 1 "1N914" V 2655 3220 50  0000 R CNN
 F 2 "Diode_THT:D_DO-35_SOD27_P7.62mm_Horizontal" H 2700 3125 50  0001 C CNN
@@
 $EndComp
 $Comp
-L Device:CP1 C?
+L Device:CP1 C1
 U 1 1 5F98CBFD
 P 2700 3800
-F 0 "C?" H 2815 3846 50  0000 L CNN
+F 0 "C1" H 2815 3846 50  0000 L CNN
 F 1 "1000uF" H 2815 3755 50  0000 L CNN
 F 2 "" H 2700 3800 50  0001 C CNN
@@
 BATTERY -
 $Comp
-L Diode:1N4004 D?
+L Diode:1N4004 D2
 U 1 1 5F98E75F
 P 4850 3250
-F 0 "D?" V 4804 3330 50  0000 L CNN
+F 0 "D2" V 4804 3330 50  0000 L CNN
 F 1 "1N4004" V 4895 3330 50  0000 L CNN
 F 2 "Diode_THT:D_DO-41_SOD81_P10.16mm_Horizontal" H 4850 3075 50  0001 C CNN
@@
 	4850 3500 5500 3500
 $Comp
-L Motor:Motor_DC M?
+L Motor:Motor_DC M1
 U 1 1 5F98FEF6
 P 6650 3000
-F 0 "M?" H 6808 2996 50  0000 L CNN
+F 0 "M1" H 6808 2996 50  0000 L CNN
 F 1 "Motor_DC" H 6808 2905 50  0000 L CNN
 F 2 "" H 6650 2910 50  0001 C CNN
@@
 Text Notes 2300 2850 0    50   ~ 0
 Diode + Cap is used\nto keep timer powered when \nmotor starts and drags down \nvoltage below 6V
-Text Notes 3750 3350 0    50   ~ 0
+Text Notes 4450 2850 0    50   ~ 0
 Flyback diode to supress\nkickback voltage when \nmotor is turned off.
 Text Notes 1650 3400 0    50   ~ 0
@@
 http://timers.shop\nTurn switch on, and apply power to configure\ndevice. Blue light should light momentarily.\nConnect to new WiFi network\nand then open http://192.168.4.1\nin browser. You may have to disable\ncellular data on your phone first.\nUse timer function #6 (repeat cycle\noff 1st). After configuration, turn switch off\nand cycle power.
 $Comp
-L Switch:SW_SPST SW?
+L Switch:SW_SPST SW1
 U 1 1 5F996FF6
 P 2800 4450
-F 0 "SW?" V 2846 4362 50  0000 R CNN
+F 0 "SW1" V 2846 4362 50  0000 R CNN
 F 1 "SW_SPST" V 2755 4362 50  0000 R CNN
 F 2 "" H 2800 4450 50  0001 C CNN
@@
 Wire Wire Line
 	3350 4250 3500 4250
+Text Notes 2900 3250 0    50   ~ 0
+use schottkey diode here \nif running from 6V lead acid\nbattery
+Text Notes 5050 4350 0    50   ~ 0
+WiFi Timer is rated from 6-28V. 6V seems \nto be the absolute min -- it will not sink \nmuch curernt unless voltage at timer is \n6V or higher.
 $EndSCHEMATC
