File: schematics/817-opto-isolator-module.kicad_sch (KiCad schematic)
At the start: 7 parts

Commit message: update 817 schematic
Parts:
- D?: V  (none) -> 1.9V @ 3mA
Other:
- note added: "1.3V @ 3mA"
- note added: "CTR ≈ 100% 3mA max output drive at 12V input"
- note added: "G"
- note added: "IN1"
- note added: "Input current = 3mA @ 12V"
- note added: "V1"
Changed lines of the file:
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@@
     (stroke (width 0) (type default) (color 0 0 0 0))
   )
-  (wire (pts (xy 127.635 74.93) (xy 135.89 74.93))
+  (wire (pts (xy 121.285 74.93) (xy 135.89 74.93))
     (stroke (width 0) (type default) (color 0 0 0 0))
   )
@@
     (stroke (width 0) (type default) (color 0 0 0 0))
   )
-  (wire (pts (xy 128.905 77.47) (xy 128.905 78.74))
+  (wire (pts (xy 122.555 77.47) (xy 122.555 78.74))
     (stroke (width 0) (type default) (color 0 0 0 0))
   )
-  (wire (pts (xy 127.635 77.47) (xy 128.905 77.47))
+  (wire (pts (xy 121.285 77.47) (xy 122.555 77.47))
     (stroke (width 0) (type default) (color 0 0 0 0))
   )
@@
   (wire (pts (xy 160.02 77.47) (xy 161.925 77.47))
     (stroke (width 0) (type default) (color 0 0 0 0))
+  )
+  (text "1.3V @ 3mA" (at 125.222 77.978 0)
+    (effects (font (size 1.27 1.27)) (justify left bottom))
+  )
+  (text "G" (at 112.522 78.486 0)
+    (effects (font (size 1.27 1.27)) (justify left bottom))
+  )
+  (text "IN1" (at 110.998 75.946 0)
+    (effects (font (size 1.27 1.27)) (justify left bottom))
+  )
+  (text "Input current = 3mA\n@ 12V" (at 119.126 72.898 0)
+    (effects (font (size 1.27 1.27)) (justify left bottom))
+  )
+  (text "G" (at 169.418 78.74 0)
+    (effects (font (size 1.27 1.27)) (justify left bottom))
+  )
+  (text "CTR ≈ 100%\n3mA max output\ndrive at 12V input" (at 173.736 78.994 0)
+    (effects (font (size 1.27 1.27)) (justify left bottom))
+  )
+  (text "V1" (at 169.164 75.946 0)
+    (effects (font (size 1.27 1.27)) (justify left bottom))
   )
   (symbol (lib_id "Jumper:Jumper_2_Open") (at 158.115 85.725 90) (unit 1)
@@
     (pin "1")
   )
-  (symbol (lib_name "Screw_Terminal_01x02_1") (lib_id "Connector:Screw_Terminal_01x02") (at 122.555 74.93 0) (mirror y) (unit 1)
+  (symbol (lib_name "Screw_Terminal_01x02_1") (lib_id "Connector:Screw_Terminal_01x02") (at 116.205 74.93 0) (mirror y) (unit 1)
     (in_bom yes) (on_board yes) (fields_autoplaced)
-    (property "Reference" "J?" (id 0) (at 122.555 83.82 0)
+    (property "Reference" "J?" (id 0) (at 116.205 83.82 0)
       (effects (font (size 1.27 1.27)) hide)
     )
-    (property "Value" "Screw_Terminal_01x02" (id 1) (at 122.555 81.28 0)
+    (property "Value" "Screw_Terminal_01x02" (id 1) (at 116.205 81.28 0)
       (effects (font (size 1.27 1.27)) hide)
     )
-    (property "Footprint" "" (id 2) (at 122.555 74.93 0)
+    (property "Footprint" "" (id 2) (at 116.205 74.93 0)
       (effects (font (size 1.27 1.27)) hide)
     )
-    (property "Datasheet" "~" (id 3) (at 122.555 74.93 0)
+    (property "Datasheet" "~" (id 3) (at 116.205 74.93 0)
       (effects (font (size 1.27 1.27)) hide)
     )
@@
     (pin "2")
   )
-  (symbol (lib_id "power:GND") (at 128.905 78.74 0) (unit 1)
+  (symbol (lib_id "power:GND") (at 122.555 78.74 0) (unit 1)
     (in_bom yes) (on_board yes) (fields_autoplaced)
-    (property "Reference" "#PWR?" (id 0) (at 128.905 85.09 0)
+    (property "Reference" "#PWR?" (id 0) (at 122.555 85.09 0)
       (effects (font (size 1.27 1.27)) hide)
     )
-    (property "Value" "GND" (id 1) (at 128.905 83.82 0))
-    (property "Footprint" "" (id 2) (at 128.905 78.74 0)
+    (property "Value" "GND" (id 1) (at 122.555 83.82 0))
+    (property "Footprint" "" (id 2) (at 122.555 78.74 0)
       (effects (font (size 1.27 1.27)) hide)
     )
-    (property "Datasheet" "" (id 3) (at 128.905 78.74 0)
+    (property "Datasheet" "" (id 3) (at 122.555 78.74 0)
       (effects (font (size 1.27 1.27)) hide)
     )
@@
       (effects (font (size 1.27 1.27)) hide)
     )
+    (property "V " "1.9V @ 3mA" (id 4) (at 125.095 92.71 90))
     (pin "1")
     (pin "2")
